File: boards/template-2layer.sch (EAGLE design)
At the start: 13 parts, among them U2 XBEE-1B3, U3 V_REG_LDOSMD

Commit message: original files from sparkfun
Parts:
- added LED1, LED2: Red, SparkFun:LED0603
- added LED3, LED4: Green, SparkFun:LED0603
- added R1, R11, R3, R4: 1K, SparkFun:RESISTOR0402-RES
- added SJ1: SOLDERJUMPERNO, SparkFun:SOLDERJUMPERNO
- added U$10, U$11, U$5, U$9: STAND-OFF, SparkFun:STAND-OFF
Connections:
- new net N$1: LED2.A, R1.2
- new net N$2: LED4.A, R4.1
- new net N$38: LED1.A, R11.1
- new net N$4: LED3.A, R3.2
- net 3.3V: now also R1.1, R11.2, R3.1
- net DIN: now also LED3.C
- net DIO3: now also SJ1.2
- net DOUT: now also LED2.C
- net GND: now also LED1.C, LED4.C
- net RSSI: now also R4.2
- net RTS: now also SJ1.1
Changed lines of the file:
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@@
 <parts>
 <part name="FRAME1" library="SparkFun" deviceset="FRAME-LETTER" device=""/>
+<part name="R11" library="SparkFun" deviceset="RESISTOR" device="0402-RES" value="1K"/>
+<part name="LED1" library="SparkFun" deviceset="LED" device="0603" value="Red"/>
+<part name="GND28" library="SparkFun" deviceset="GND" device=""/>
+<part name="LED2" library="SparkFun" deviceset="LED" device="0603" value="Red"/>
+<part name="LED3" library="SparkFun" deviceset="LED" device="0603" value="Green"/>
+<part name="R1" library="SparkFun" deviceset="RESISTOR" device="0402-RES" value="1K"/>
+<part name="R3" library="SparkFun" deviceset="RESISTOR" device="0402-RES" value="1K"/>
 <part name="U$7" library="SparkFun" deviceset="FIDUCIAL" device="1X2"/>
 <part name="U$16" library="SparkFun" deviceset="FIDUCIAL" device="1X2"/>
@@
 <part name="P+1" library="SparkFun" deviceset="3.3V" device=""/>
 <part name="GND2" library="SparkFun" deviceset="GND" device=""/>
+<part name="U$5" library="SparkFun" deviceset="STAND-OFF" device=""/>
+<part name="U$9" library="SparkFun" deviceset="STAND-OFF" device=""/>
+<part name="U$10" library="SparkFun" deviceset="STAND-OFF" device=""/>
+<part name="U$11" library="SparkFun" deviceset="STAND-OFF" device=""/>
+<part name="LED4" library="SparkFun" deviceset="LED" device="0603" value="Green"/>
+<part name="R4" library="SparkFun" deviceset="RESISTOR" device="0402-RES" value="1K"/>
+<part name="GND4" library="SparkFun" deviceset="GND" device=""/>
 <part name="U3" library="SparkFun" deviceset="V_REG_LDO" device="SMD"/>
 <part name="GND1" library="SparkFun" deviceset="GND" device=""/>
@@
 <part name="C3" library="SparkFun" deviceset="CAP_POL" device="1206" value="10uF"/>
 <part name="GND6" library="SparkFun" deviceset="GND" device=""/>
+<part name="P+2" library="SparkFun" deviceset="3.3V" device=""/>
+<part name="SJ1" library="SparkFun" deviceset="SOLDERJUMPER" device="NO"/>
 <part name="JP4" library="SparkFun" deviceset="ARDUINO_SERIAL_PROGRAM" device="PTH"/>
 <part name="D1" library="SparkFun" deviceset="DIODE" device="SOD"/>
+<part name="P+3" library="SparkFun" deviceset="3.3V" device=""/>
+<part name="P+4" library="SparkFun" deviceset="3.3V" device=""/>
 </parts>
 <sheets>
@@
 <instance part="FRAME1" gate="G$1" x="0" y="0"/>
 <instance part="FRAME1" gate="G$2" x="147.32" y="0"/>
+<instance part="R11" gate="G$1" x="63.5" y="45.72" rot="R90"/>
+<instance part="LED1" gate="G$1" x="63.5" y="35.56"/>
+<instance part="GND28" gate="1" x="63.5" y="25.4"/>
+<instance part="LED2" gate="G$1" x="27.94" y="38.1"/>
+<instance part="LED3" gate="G$1" x="38.1" y="38.1"/>
+<instance part="R1" gate="G$1" x="27.94" y="48.26" rot="R270"/>
+<instance part="R3" gate="G$1" x="38.1" y="48.26" rot="R270"/>
 <instance part="U$7" gate="G$1" x="243.84" y="27.94"/>
 <instance part="U$16" gate="G$1" x="238.76" y="27.94"/>
@@
 <instance part="P+1" gate="G$1" x="99.06" y="116.84"/>
 <instance part="GND2" gate="1" x="99.06" y="86.36"/>
+<instance part="U$5" gate="G$1" x="233.68" y="27.94"/>
+<instance part="U$9" gate="G$1" x="228.6" y="27.94"/>
+<instance part="U$10" gate="G$1" x="223.52" y="27.94"/>
+<instance part="U$11" gate="G$1" x="218.44" y="27.94"/>
+<instance part="LED4" gate="G$1" x="50.8" y="35.56"/>
+<instance part="R4" gate="G$1" x="50.8" y="45.72" rot="R90"/>
+<instance part="GND4" gate="1" x="50.8" y="25.4"/>
 <instance part="U3" gate="G$1" x="121.92" y="157.48"/>
 <instance part="GND1" gate="1" x="106.68" y="147.32"/>
@@
 <instance part="C3" gate="G$1" x="99.06" y="157.48"/>
 <instance part="GND6" gate="1" x="99.06" y="147.32"/>
+<instance part="P+2" gate="G$1" x="63.5" y="53.34"/>
+<instance part="SJ1" gate="1" x="121.92" y="50.8"/>
 <instance part="JP4" gate="G$1" x="27.94" y="104.14" rot="MR180"/>
 <instance part="D1" gate="G$1" x="96.52" y="109.22" rot="R180"/>
+<instance part="P+3" gate="G$1" x="38.1" y="55.88"/>
+<instance part="P+4" gate="G$1" x="27.94" y="55.88"/>
 </instances>
 <busses>
@@
 <nets>
 <net name="GND" class="1">
+<segment>
+<wire x1="63.5" y1="30.48" x2="63.5" y2="27.94" width="0.1524" layer="91"/>
+<pinref part="LED1" gate="G$1" pin="C"/>
+<pinref part="GND28" gate="1" pin="GND"/>
+</segment>
 <segment>
 <wire x1="101.6" y1="91.44" x2="99.06" y2="91.44" width="0.1524" layer="91"/>
@@
 <pinref part="GND2" gate="1" pin="GND"/>
 <pinref part="JP2" gate="G$1" pin="1"/>
+</segment>
+<segment>
+<wire x1="50.8" y1="30.48" x2="50.8" y2="27.94" width="0.1524" layer="91"/>
+<pinref part="LED4" gate="G$1" pin="C"/>
+<pinref part="GND4" gate="1" pin="GND"/>
 </segment>
 <segment>
@@
 </segment>
 </net>
+<net name="N$38" class="0">
+<segment>
+<wire x1="63.5" y1="38.1" x2="63.5" y2="40.64" width="0.1524" layer="91"/>
+<pinref part="R11" gate="G$1" pin="1"/>
+<pinref part="LED1" gate="G$1" pin="A"/>
+</segment>
+</net>
+<net name="N$1" class="0">
+<segment>
+<wire x1="27.94" y1="43.18" x2="27.94" y2="40.64" width="0.1524" layer="91"/>
+<pinref part="LED2" gate="G$1" pin="A"/>
+<pinref part="R1" gate="G$1" pin="2"/>
+</segment>
+</net>
+<net name="N$4" class="0">
+<segment>
+<wire x1="38.1" y1="43.18" x2="38.1" y2="40.64" width="0.1524" layer="91"/>
+<pinref part="LED3" gate="G$1" pin="A"/>
+<pinref part="R3" gate="G$1" pin="2"/>
+</segment>
+</net>
 <net name="DIN" class="0">
 <segment>
@@
 </segment>
 <segment>
+<wire x1="38.1" y1="33.02" x2="38.1" y2="25.4" width="0.1524" layer="91"/>
+<label x="38.1" y="25.4" size="1.778" layer="95" rot="R90"/>
+<pinref part="LED3" gate="G$1" pin="C"/>
+</segment>
+<segment>
 <wire x1="33.02" y1="106.68" x2="40.64" y2="106.68" width="0.1524" layer="91"/>
 <label x="35.56" y="106.68" size="1.778" layer="95"/>
@@
 <pinref part="U2" gate="G$1" pin="DOUT"/>
 <pinref part="JP2" gate="G$1" pin="9"/>
+</segment>
+<segment>
+<wire x1="27.94" y1="33.02" x2="27.94" y2="25.4" width="0.1524" layer="91"/>
+<label x="27.94" y="25.4" size="1.778" layer="95" rot="R90"/>
+<pinref part="LED2" gate="G$1" pin="C"/>
 </segment>
 <segment>
@@
 <pinref part="C2" gate="G$1" pin="1"/>
 </segment>
+<segment>
+<wire x1="63.5" y1="53.34" x2="63.5" y2="50.8" width="0.1524" layer="91"/>
+<pinref part="R11" gate="G$1" pin="2"/>
+<pinref part="P+2" gate="G$1" pin="3.3V"/>
+</segment>
+<segment>
+<wire x1="38.1" y1="53.34" x2="38.1" y2="55.88" width="0.1524" layer="91"/>
+<pinref part="R3" gate="G$1" pin="1"/>
+<pinref part="P+3" gate="G$1" pin="3.3V"/>
+</segment>
+<segment>
+<wire x1="27.94" y1="53.34" x2="27.94" y2="55.88" width="0.1524" layer="91"/>
+<pinref part="R1" gate="G$1" pin="1"/>
+<pinref part="P+4" gate="G$1" pin="3.3V"/>
+</segment>
 </net>
 <net name="DIO4" class="0">
@@
 <pinref part="JP3" gate="G$1" pin="5"/>
 </segment>
+<segment>
+<wire x1="116.84" y1="50.8" x2="109.22" y2="50.8" width="0.1524" layer="91"/>
+<label x="109.22" y="50.8" size="1.778" layer="95"/>
+<pinref part="SJ1" gate="1" pin="1"/>
+</segment>
 </net>
 <net name="DIO3" class="0">
@@
 </segment>
 <segment>
+<wire x1="127" y1="50.8" x2="134.62" y2="50.8" width="0.1524" layer="91"/>
+<label x="129.54" y="50.8" size="1.778" layer="95"/>
+<pinref part="SJ1" gate="1" pin="2"/>
+</segment>
+<segment>
 <wire x1="33.02" y1="109.22" x2="40.64" y2="109.22" width="0.1524" layer="91"/>
 <label x="35.56" y="109.22" size="1.778" layer="95"/>
@@
 <pinref part="JP2" gate="G$1" pin="5"/>
 </segment>
+<segment>
+<wire x1="50.8" y1="50.8" x2="50.8" y2="58.42" width="0.1524" layer="91"/>
+<label x="50.8" y="53.34" size="1.778" layer="95" rot="R90"/>
+<pinref part="R4" gate="G$1" pin="2"/>
+</segment>
 </net>
 <net name="DIO12" class="0">
@@
 </segment>
 </net>
+<net name="N$2" class="0">
+<segment>
+<wire x1="50.8" y1="40.64" x2="50.8" y2="38.1" width="0.1524" layer="91"/>
+<pinref part="LED4" gate="G$1" pin="A"/>
+<pinref part="R4" gate="G$1" pin="1"/>
+</segment>
+</net>

Commit message: cleaned up template
Parts:
- removed C1, C3: 10uF, SparkFun:CAP_POL1206
- removed C2: 0.1uF, SparkFun:CAP0402-CAP
- removed D1: (no value), SparkFun:DIODESOD
- removed JP2, JP3: M11PTH, SparkFun:M11PTH
- removed JP4: (no value), SparkFun:ARDUINO_SERIAL_PROGRAMPTH
- removed LED1, LED2: Red, SparkFun:LED0603
- removed LED3, LED4: Green, SparkFun:LED0603
- removed R1, R11, R3, R4: 1K, SparkFun:RESISTOR0402-RES
- removed SJ1: SOLDERJUMPERNO, SparkFun:SOLDERJUMPERNO
- removed U$1: LOGO-SFESK, SparkFun:LOGO-SFESK
- removed U$10, U$11, U$5, U$9: STAND-OFF, SparkFun:STAND-OFF
- removed U$16, U$7: FIDUCIAL1X2, SparkFun:FIDUCIAL1X2
- removed U$4: LOGO-SFENEW, SparkFun:LOGO-SFENEW
- removed U3: V_REG_LDOSMD, SparkFun:V_REG_LDOSMD
Connections:
- removed net 5V: C3.+, JP3.11, JP4.VCC, U3.EN, U3.IN
- removed net DIN: D1.C, JP2.8, JP4.RXI, LED3.C
- removed net N$1: LED2.A, R1.2
- removed net N$2: LED4.A, R4.1
- removed net N$3: D1.A, U2.DIN
- removed net N$38: LED1.A, R11.1
- removed net N$4: LED3.A, R3.2
- net 3.3V: no longer C1.+, C2.1, JP2.10, R1.1, R11.2, R3.1, U3.OUT
- net CTS: no longer JP3.9
- net DIO0: no longer JP3.1
- net DIO1: no longer JP3.2
- net DIO11: no longer JP2.4
- net DIO12: no longer JP2.7
- net DIO2: no longer JP3.3
- net DIO3: no longer JP3.4, JP4.DTR, SJ1.2
- net DIO4: no longer JP3.10
- net DIO5: no longer JP3.6
- net DIO9: no longer JP3.8
- net DOUT: no longer JP2.9, JP4.TXO, LED2.C
- net DTR: no longer JP2.2
- net GND: no longer C1.-, C2.2, C3.-, JP2.1, JP2.11, JP4.CTS, JP4.GND, LED1.C, LED4.C, U3.GND
- net RES1: no longer JP2.3
- net RES2: no longer JP3.7
- net RESET: no longer JP2.6
- net RSSI: no longer JP2.5, R4.2
- net RTS: no longer JP3.5, SJ1.1
